Commit message: stage2

File: dev_ws/src/test3d_ros/description/robot_core.xacro (robot description, xacro)
@@ -1,7 +1,7 @@
 <?xml version="1.0"?>
 <robot xmlns:xacro="http://www.ros.org/wiki/xacro" >
-    <xacro:include filename="inertial_macros.xacro" />
+    <xacro:include filename="inertial_macros.xacro"/>
     <material name="white">
-        <color rgba="1 1 1 1"/>
+        <color rgba="1 1 1 1" />
     </material>
     <material name="orange">
@@ -25,5 +25,5 @@
     <link name="chassis">
         <visual>
-            <origin xyz="0.15 0 0.075" rpy="0 0 0"/>
+            <origin xyz="0.15 0 0.075"/>
             <geometry>
                 <box size="0.3 0.3 0.15"/>
@@ -31,19 +31,22 @@
             <material name="white"/>
         </visual>
-        <colllision>
-            <origin xyz="0.15 0 0.075" rpy="0 0 0"/>
+        <collision>
+            <origin xyz="0.15 0 0.075"/>
             <geometry>
                 <box size="0.3 0.3 0.15"/>
             </geometry>
-        </colllision>
+        </collision>
         <xacro:inertial_box mass="0.5" x="0.3" y="0.3" z="0.15">
             <origin xyz="0.15 0 0.075" rpy="0 0 0"/>
         </xacro:inertial_box>
     </link>
-    <!-- LEFT WHEEL -->
+    <gazebo reference="chassis">
+        <material>Gazebo/White</material>
+    </gazebo>
+    <!-- LEFT WHEEL LINK -->
     <joint name="left_wheel_joint" type="continuous">
         <parent link="base_link"/>
         <child link="left_wheel"/>
-        <origin xyz="0 0.175 0" rpy="-${pi/2} 0 0"/>
+        <origin xyz="0 0.175 0" rpy="-${pi/2} 0 0" />
         <axis xyz="0 0 1"/>
     </joint>
@@ -51,22 +54,25 @@
         <visual>
             <geometry>
-                <cylinder length="0.04" radius="0.05" />/>
+                <cylinder radius="0.05" length="0.04"/>
             </geometry>
             <material name="blue"/>
         </visual>
-        <colllision>
+        <collision>
             <geometry>
-                <cylinder length="0.04" radius="0.05" />/>
+                <cylinder radius="0.05" length="0.04"/>
             </geometry>
-        </colllision>
-        <xacro:inertial_cylinder mass="0.1" length="0.05" radius="0.05">
+        </collision>
+        <xacro:inertial_cylinder mass="0.1" length="0.04" radius="0.05">
             <origin xyz="0 0 0" rpy="0 0 0"/>
         </xacro:inertial_cylinder>
     </link>
-    <!-- RIGHT WHEEL -->
+    <gazebo reference="left_wheel">
+        <material>Gazebo/Blue</material>
+    </gazebo>
+    <!-- RIGHT WHEEL LINK -->
     <joint name="right_wheel_joint" type="continuous">
         <parent link="base_link"/>
         <child link="right_wheel"/>
-        <origin xyz="0 -0.175 0" rpy="${pi/2} 0 0"/>
+        <origin xyz="0 -0.175 0" rpy="${pi/2} 0 0" />
         <axis xyz="0 0 -1"/>
     </joint>
@@ -74,38 +80,46 @@
         <visual>
             <geometry>
-                <cylinder length="0.04" radius="0.05" />/>
+                <cylinder radius="0.05" length="0.04"/>
             </geometry>
             <material name="blue"/>
         </visual>
-        <colllision>
+        <collision>
             <geometry>
-                <cylinder length="0.04" radius="0.05" />/>
+                <cylinder radius="0.05" length="0.04"/>
             </geometry>
-        </colllision>
-        <xacro:inertial_cylinder mass="0.1" length="0.05" radius="0.05">
+        </collision>
+        <xacro:inertial_cylinder mass="0.1" length="0.04" radius="0.05">
             <origin xyz="0 0 0" rpy="0 0 0"/>
         </xacro:inertial_cylinder>
     </link>
-    <!-- CASTER WHEEL -->
+    <gazebo reference="right_wheel">
+        <material>Gazebo/Blue</material>
+    </gazebo>
+    <!-- CASTER WHEEL LINK -->
     <joint name="caster_wheel_joint" type="fixed">
         <parent link="chassis"/>
         <child link="caster_wheel"/>
-        <origin xyz="0.24 0 0" rpy="0 0 0"/>
+        <origin xyz="0.24 0 0"/>
     </joint>
     <link name="caster_wheel">
         <visual>
             <geometry>
-                <sphere radius="0.05" />
+                <sphere radius="0.05"/>
             </geometry>
             <material name="black"/>
         </visual>
-        <colllision>
+        <collision>
             <geometry>
-                <sphere radius="0.05" />
+                <sphere radius="0.05"/>
             </geometry>
-        </colllision>
+        </collision>
         <xacro:inertial_sphere mass="0.1" radius="0.05">
             <origin xyz="0 0 0" rpy="0 0 0"/>
         </xacro:inertial_sphere>
     </link>
+    <gazebo reference="caster_wheel">
+        <material>Gazebo/Black</material>
+        <mu1 value="0.001"/>
+        <mu2 value="0.001"/>
+    </gazebo>
 </robot>
